File: konoha.kicad_sch (KiCad schematic)
At the start: 72 parts, among them J1 Port_1_C, J2 Port_2_C, J3 Port_3, J4 Port_4, J5 Port_Host, J6 Port_Charge_PowerOnly, U1 CH634X, U10 TPD4E02B04DQA, U11 TPD4E02B04DQA, U13 TPD4E02B04DQA, U14 USBLC6-2P6, U15 CH213K, U16 CH217K, U17 CH217K, U18 CH217K, U19 CH217K, U2 TPD4E02B04DQA, U5 TPD4E02B04DQA, U6 TPD4E02B04DQA, U7 TPD4E02B04DQA, Y1 24MHz

Commit message: v2 schematic and board
Parts:
- removed C32, C33, C34: 0.1uF, Capacitor_SMD:C_0402_1005Metric_Pad0.74x0.62mm_HandSolder, symbol Device:C_Small
- removed J2: Port_2_C, footprint:USB-C-SMD_TYPE-C-24P-QT, symbol Connector:USB_C_Receptacle
- removed U10, U2: TPD4E02B04DQA, Package_SON:USON-10_2.5x1.0mm_P0.5mm, symbol Power_Protection:TPD4E02B04DQA
- removed U14: USBLC6-2P6, Package_TO_SOT_SMD:SOT-666, symbol Power_Protection:USBLC6-2P6
- added C35, C36, C37, C38, C39, C40: 0.1uF, Capacitor_SMD:C_0603_1608Metric_Pad1.08x0.95mm_HandSolder, symbol Device:C_Small
- added C41, C42: 1uF, Capacitor_SMD:C_0603_1608Metric_Pad1.08x0.95mm_HandSolder, symbol Device:C_Small
- added D3: SMAJ5.0CA, Diode_SMD:D_SMA, symbol Diode:SMAJ5.0CA
- added J1: Port_1, footprint:TYPE-C-USB-SMD_QCHT-143, symbol Connector:USB_C_Receptacle
- added R15, R18, R20: 500K, Resistor_SMD:R_0603_1608Metric_Pad0.98x0.95mm_HandSolder, symbol Device:R_Small
- added R16, R17, R19: 200K, Resistor_SMD:R_0603_1608Metric_Pad0.98x0.95mm_HandSolder, symbol Device:R_Small
- added R21, R22: 5.1K, Resistor_SMD:R_0603_1608Metric_Pad0.98x0.95mm_HandSolder, symbol Device:R_Small
- added R23: 10K, Resistor_SMD:R_0603_1608Metric_Pad0.98x0.95mm_HandSolder, symbol Device:R_Small
- added U10: WS3202E61-6/TR, footprint:SOT-23-6_L2.9-W1.6-P0.95-LS2.8-BR, symbol WS3202E61-6TR:WS3202E61-6/TR
- added U12, U14, U25, U26, U8, U9: TPD4E02B04DQA, Package_SON:USON-10_2.5x1.0mm_P0.5mm, symbol Power_Protection:TPD4E02B04DQA
- added U2, U3, U4: HD3SS3220IRNHR, Package_DFN_QFN:Texas_RNH0030A_WQFN-30-1EP_2.5x4.5mm_P0.4mm_EP1.2x3.2mm_ThermalVias, symbol HD3SS3220RNH:HD3SS3220IRNHR
- added U20, U21, U22, U23, U24: USBLC6-2SC6, Package_TO_SOT_SMD:SOT-23-6, symbol Power_Protection:USBLC6-2SC6
- C1, C10, C11, C12, C13, C14, C15, C2, C21, C22, C23, C24, C25, C26, C27, C28, C3, C4, C5, C6, C7, C8, C9: footprint Capacitor_SMD:C_0402_1005Metric_Pad0.74x0.62mm_HandSolder -> Capacitor_SMD:C_0603_1608Metric_Pad1.08x0.95mm_HandSolder
- C16: footprint Capacitor_THT:CP_Radial_D10.0mm_P5.00mm -> Capacitor_SMD:CP_Elec_6.3x7.7
- C29: value 0.1uF -> 100uF; footprint Capacitor_SMD:C_0402_1005Metric_Pad0.74x0.62mm_HandSolder -> Capacitor_SMD:C_1206_3216Metric
- C30: value 0.1uF -> 100nF; footprint Capacitor_SMD:C_0402_1005Metric_Pad0.74x0.62mm_HandSolder -> Capacitor_SMD:C_0603_1608Metric_Pad1.08x0.95mm_HandSolder
- C31: value 0.1uF -> 470uF; footprint Capacitor_SMD:C_0402_1005Metric_Pad0.74x0.62mm_HandSolder -> Capacitor_SMD:CP_Elec_6.3x7.7
- D1: now not fitted
- J2: renamed from J1; value Port_1_C -> Port_2; footprint footprint:USB-C-SMD_TYPE-C-24P-QT -> footprint:TYPE-C-USB-SMD_QCHT-143
- J3, J4, J5: footprint footprint:USB-C-SMD_TYPE-C-24P-QT -> footprint:TYPE-C-USB-SMD_QCHT-143
- R1: footprint Resistor_SMD:R_0402_1005Metric_Pad0.72x0.64mm_HandSolder -> Resistor_SMD:R_0603_1608Metric_Pad0.98x0.95mm_HandSolder; now not fitted
- R10, R12: value 5.1K -> 200K; footprint Resistor_SMD:R_0402_1005Metric_Pad0.72x0.64mm_HandSolder -> Resistor_SMD:R_0603_1608Metric_Pad0.98x0.95mm_HandSolder
- R11, R9: value 5.1K -> 900K; footprint Resistor_SMD:R_0402_1005Metric_Pad0.72x0.64mm_HandSolder -> Resistor_SMD:R_0603_1608Metric_Pad0.98x0.95mm_HandSolder
- R13: value 56K -> 900K; footprint Resistor_SMD:R_0402_1005Metric_Pad0.72x0.64mm_HandSolder -> Resistor_SMD:R_0603_1608Metric_Pad0.98x0.95mm_HandSolder
- R14: value 56K -> 200K; footprint Resistor_SMD:R_0402_1005Metric_Pad0.72x0.64mm_HandSolder -> Resistor_SMD:R_0603_1608Metric_Pad0.98x0.95mm_HandSolder
- R2, R3, R4: footprint Resistor_SMD:R_0402_1005Metric_Pad0.72x0.64mm_HandSolder -> Resistor_SMD:R_0603_1608Metric_Pad0.98x0.95mm_HandSolder
- R5, R6, R7, R8: value 24K -> 30K; footprint Resistor_SMD:R_0402_1005Metric_Pad0.72x0.64mm_HandSolder -> Resistor_SMD:R_0603_1608Metric_Pad0.98x0.95mm_HandSolder
- U11, U13, U5, U6, U7: now fitted; now in the parts list
Connections:
- net +3V3: now also R10.2, R12.2, R14.2, R23.2, U2.8 (VCC33), U3.8 (VCC33), U4.8 (VCC33); no longer U1.27 (OVCUR1#), U1.29 (OVCUR2#), U1.31 (OVCUR3#/GANG_EN#), U1.33 (OVCUR4#/GANG_EN#), U1.46 (RESET#), U16.3 (FLAG#), U17.3 (FLAG#), U18.3 (FLAG#), U19.3 (FLAG#)
- net +5V: now also C31.2, C42.2, D3.1 (A1), U10.4 (OUT); no longer J6.A9 (VBUS), J6.B9 (VBUS)
- net +5VD: now also C18.1, R15.2, R16.2, R17.2, R18.2, R19.2, R20.2, U2.30 (VDD5), U21.5 (VBUS), U3.30 (VDD5), U4.30 (VDD5)
- net GND: now also C29.2, C30.2, C31.1, C41.1, C42.1, D3.2 (A2), J1.A1 (GND), J1.A12 (GND), J1.B1 (GND), J1.B12 (GND), R21.2, R22.2, U10.1 (GND), U10.2 (GND), U10.5 (GND), U10.6 (GND), U12.3 (G), U12.8 (G), U14.3 (G), U14.8 (G), U2.12 (EN_MUX_N), U2.13 (GND), U2.28 (GND), U2.29 (EN_CC_N), U2.31 (PAD), U20.2 (GND), U21.2 (GND), U22.2 (GND), U23.2 (GND), U24.2 (GND), U25.3 (G), U25.8 (G), U26.3 (G), U26.8 (G), U3.12 (EN_MUX_N), U3.13 (GND), U3.28 (GND), U3.29 (EN_CC_N), U3.31 (PAD), U4.12 (EN_MUX_N), U4.13 (GND), U4.28 (GND), U4.29 (EN_CC_N), U4.31 (PAD), U8.3 (G), U8.8 (G), U9.3 (G), U9.8 (G); no longer J2.S1 (SHIELD), J3.S1 (SHIELD), J4.S1 (SHIELD), J5.S1 (SHIELD), J6.S1 (SHIELD), R10.2, R11.2, R12.2, R13.2, R14.2, R9.2
- net P1C_SS_RX+: now also J5.A11 (RX2+), U13.2 (IO2); no longer J2.A11 (RX2+), U6.4 (IO3)
- net P1C_SS_RX-: now also J5.A10 (RX2-), U13.1 (IO1); no longer J2.A10 (RX2-), U6.5 (IO4)
- net P1C_SS_TX+: now also C26.2; no longer C24.2, U6.1 (IO1)
- net P1C_SS_TX-: now also C25.2; no longer C23.2, U6.2 (IO2)
- net P1_CC1: now also J5.A5 (CC1), R21.1; no longer J2.A5 (CC1)
- net P1_CC2: now also J5.B5 (CC2), R22.1; no longer J2.B5 (CC2)
- net P1_HS_D+: now also U21.4 (I/O2); no longer J2.A6 (D+)
- net P1_HS_D-: now also U21.6 (I/O1); no longer J2.A7 (D-)
- net P1_SS_RX+: now also J5.B11 (RX1+), U1.55 (P1_SS_RXA), U12.2 (IO2); no longer J2.B11 (RX1+), U1.56 (P1_SS_RXB)
- net P1_SS_RX-: now also J5.B10 (RX1-), U1.56 (P1_SS_RXB), U12.1 (IO1); no longer J2.B10 (RX1-), U1.55 (P1_SS_RXA)
- net P1_SS_TX+: now also C28.2; no longer C22.2
- net P1_SS_TX-: now also C27.2; no longer C21.2
- net P2C_SS_RX+: now also J2.A11 (RX2+), U11.2 (IO2); no longer U7.4 (IO3)
- net P2C_SS_RX-: now also J2.A10 (RX2-), U11.1 (IO1); no longer U7.5 (IO4)
- net P2C_SS_TX+: now also C24.2; no longer C28.2, U7.1 (IO1)
- net P2C_SS_TX-: now also C23.2; no longer C27.2, U7.2 (IO2)
- net P2_CC1: now also J2.A5 (CC1)
- net P2_CC2: now also J2.B5 (CC2)
- net P2_HS_D+: now also U20.4 (I/O2)
- net P2_HS_D-: now also U20.6 (I/O1)
- net P2_SS_RX+: now also J2.B11 (RX1+), U9.2 (IO2); no longer U5.4 (IO3)
- net P2_SS_RX-: now also J2.B10 (RX1-), U9.1 (IO1); no longer U5.5 (IO4)
- net P2_SS_TX+: now also C22.2; no longer C26.2, U5.1 (IO1)
- net P2_SS_TX-: now also C21.2; no longer C25.2, U5.2 (IO2)
- net P3_HS_D+: now also U23.4 (I/O2); no longer J3.A6 (D+)
- net P3_HS_D-: now also U23.6 (I/O1); no longer J3.A7 (D-)
- net P3_SS_RX+: now also U1.14 (P3_SS_RXA), U3.9 (RXP); no longer J3.B11 (RX1+), U1.13 (P3_SS_RXB)
- net P3_SS_RX-: now also U1.13 (P3_SS_RXB), U3.10 (RXN); no longer J3.B10 (RX1-), U1.14 (P3_SS_RXA)
- net P3_SS_TX+: now also U1.11 (P3_SS_TXA), C35.2; no longer C30.2, U1.10 (P3_SS_TXB)
- net P3_SS_TX-: now also U1.10 (P3_SS_TXB), C36.2; no longer C29.2, U1.11 (P3_SS_TXA)
- net P4_HS_D+: now also U24.4 (I/O2); no longer J4.A6 (D+)
- net P4_HS_D-: now also U24.6 (I/O1); no longer J4.A7 (D-)
- net P4_SS_RX+: now also U1.5 (P4_SS_RXA), U4.9 (RXP); no longer J4.B11 (RX1+), U1.4 (P4_SS_RXB), U11.4 (IO3)
- net P4_SS_RX-: now also U1.4 (P4_SS_RXB), U4.10 (RXN); no longer J4.B10 (RX1-), U1.5 (P4_SS_RXA), U11.5 (IO4)
- net P4_SS_TX+: now also U1.2 (P4_SS_TXA), C37.2; no longer U1.1 (P4_SS_TXB), U11.1 (IO1)
- net P4_SS_TX-: now also U1.1 (P4_SS_TXB), C38.2; no longer C31.2, U1.2 (P4_SS_TXA), U11.2 (IO2)
- net UP_HS_D+: now also U22.4 (I/O2); no longer J5.A6 (D+)
- net UP_HS_D-: now also U22.6 (I/O1); no longer J5.A7 (D-)
- net UP_SS_RX+: now also U14.1 (IO1), U2.10 (RXN); no longer J5.B11 (RX1+), U13.4 (IO3)
- net UP_SS_RX-: now also U14.2 (IO2), U2.9 (RXP); no longer J5.B10 (RX1-), U13.5 (IO4)
- net UP_SS_TX+: now also U1.65 (UP_SS_TXA), C39.2; no longer U1.64 (UP_SS_TXB), U13.1 (IO1)
- net UP_SS_TX-: now also U1.64 (UP_SS_TXB), C40.2; no longer U1.65 (UP_SS_TXA), U13.2 (IO2)
- net VBUS1: now also C29.1, R13.2, J1.A4 (VBUS), J1.A9 (VBUS), J1.B4 (VBUS), J1.B9 (VBUS), U22.5 (VBUS); no longer C17.1, J2.A4 (VBUS), J2.A9 (VBUS), J2.B4 (VBUS), J2.B9 (VBUS)
- net VBUS2: now also C17.1, J2.A4 (VBUS), J2.A9 (VBUS), J2.B4 (VBUS), J2.B9 (VBUS), U20.5 (VBUS); no longer C18.1
- net VBUS3: now also R9.2, U23.5 (VBUS)
- net VBUS4: now also R11.2, U24.5 (VBUS)
- net P1_SS_AC_TX-: now reaches J5.A3 (TX1-)
- net P1_SS_AC_TX-: now also C27.1, U12.4 (IO3)
- net P2C_SS_AC_TX-: now reaches C23.1, J2.B3 (TX2-)
- net P2C_SS_AC_TX-: now also U11.4 (IO3)
- net at J3.A5 (CC1): now also U3.2 (CC1); no longer R9.1
- net P1_SS_AC_TX+: now reaches C28.1
- net P1_SS_AC_TX+: now also J5.A2 (TX1+), U12.5 (IO4)
- net at J6.A5 (CC1): now also R3.1
- net at J6.B5 (CC2): now also R4.1
- net P4_SS_TX1+: now reaches J4.A2 (TX1+)
- net P4_SS_TX1+: now also U7.2 (IO2), U4.16 (TX1N)
- net at R14.1: now also U2.11 (DIR); no longer J5.B5 (CC2)
- net P3_SS_TX1+: now reaches J3.A2 (TX1+)
- net P3_SS_TX1+: now also U5.4 (IO3), U3.16 (TX1N); no longer C30.1
- net P2_SS_AC_TX-: now reaches C21.1, J2.A3 (TX1-)
- net P2_SS_AC_TX-: now also U9.4 (IO3)
- net P2_SS_AC_TX+: now reaches C22.1, J2.A2 (TX1+)
- net P2_SS_AC_TX+: now also U9.5 (IO4)
- net P2C_SS_AC_TX+: now reaches C24.1, J2.B2 (TX2+)
- net P2C_SS_AC_TX+: now also U11.5 (IO4)
- net P2_HS_AC_D+: now reaches J2.B6 (D+)
- net P2_HS_AC_D+: now also J2.A6 (D+), U20.3 (I/O2)
- net P2_HS_AC_D-: now reaches J2.B7 (D-)
- net P2_HS_AC_D-: now also J2.A7 (D-), U20.1 (I/O1)
- net at J4.B5 (CC2): now also U4.1 (CC2); no longer R12.1
- net P4_SS_TX1-: now reaches J4.A3 (TX1-)
- net P4_SS_TX1-: now also U7.1 (IO1), U4.17 (TX1P); no longer C31.1
- net P3_SS_RX2-: now reaches J3.A10 (RX2-)
- net P3_SS_RX2-: now also U6.1 (IO1), U3.18 (RX2N)
- net P3_SS_RX2+: now reaches J3.A11 (RX2+)
- net P3_SS_RX2+: now also U6.2 (IO2), U3.19 (RX2P)
- net P3_SS_TX1-: now reaches J3.A3 (TX1-)
- net P3_SS_TX1-: now also U5.5 (IO4), U3.17 (TX1P); no longer C29.1
- net P3_SS_TX2+: now reaches J3.B2 (TX2+)
- net P3_SS_TX2+: now also U6.5 (IO4), U3.21 (TX2P)
- net P3_SS_TX2-: now reaches J3.B3 (TX2-)
- net P3_SS_TX2-: now also U6.4 (IO3), U3.20 (TX2N)
- net at J3.B5 (CC2): now also U3.1 (CC2); no longer R10.1
- net P3_HS_AC_D+: now reaches J3.B6 (D+)
- net P3_HS_AC_D+: now also J3.A6 (D+), U23.3 (I/O2)
- net P3_HS_AC_D-: now reaches J3.B7 (D-)
- net P3_HS_AC_D-: now also J3.A7 (D-), U23.1 (I/O1)
- net at R13.1: now also U2.5 (VBUS_DET); no longer J5.A5 (CC1)
- net P1C_SS_AC_TX+: now reaches C26.1
- net P1C_SS_AC_TX+: now also J5.B2 (TX2+), U13.5 (IO4)
- net P1C_SS_AC_TX-: now reaches C25.1
- net P1C_SS_AC_TX-: now also J5.B3 (TX2-), U13.4 (IO3)
- net P4_SS_RX2-: now reaches J4.A10 (RX2-)
- net P4_SS_RX2-: now also U4.18 (RX2N), U8.1 (IO1)
- net P4_SS_RX2+: now reaches J4.A11 (RX2+)
- net P4_SS_RX2+: now also U4.19 (RX2P), U8.2 (IO2)
- net at R11.1: now also U4.5 (VBUS_DET); no longer J4.A5 (CC1)
- net P4_SS_TX2+: now reaches J4.B2 (TX2+)
- net P4_SS_TX2+: now also U4.21 (TX2P), U8.5 (IO4)
- net P4_SS_TX2-: now reaches J4.B3 (TX2-)
- net P4_SS_TX2-: now also U4.20 (TX2N), U8.4 (IO3)
- net P4_HS_AC_D+: now reaches J4.B6 (D+)
- net P4_HS_AC_D+: now also J4.A6 (D+), U24.3 (I/O2)
- net P4_HS_AC_D-: now reaches J4.B7 (D-)
- net P4_HS_AC_D-: now also J4.A7 (D-), U24.1 (I/O1)
- net P1_HS_AC_D+: now reaches J5.B6 (D+)
- net P1_HS_AC_D+: now also J5.A6 (D+), U21.3 (I/O2)
- net P1_HS_AC_D-: now reaches J5.B7 (D-)
- net P1_HS_AC_D-: now also J5.A7 (D-), U21.1 (I/O1)
- new net: R15.1, U3.3 (CURRENT_MODE)
- new net: J1.A5 (CC1), U2.2 (CC1)
- new net: J1.B5 (CC2), U2.1 (CC2)
- new net: R20.1, U2.3 (CURRENT_MODE)
- new net: R19.1, U2.4 (PORT)
- new net: R10.1, U3.11 (DIR)
- new net: R16.1, U3.4 (PORT)
- new net: R9.1, U3.5 (VBUS_DET)
- new net: R18.1, U4.3 (CURRENT_MODE)
- new net: C41.2, J6.A9 (VBUS), J6.B9 (VBUS), U10.3 (IN)
- new net: J4.A5 (CC1), U4.2 (CC1)
- new net: R12.1, U4.11 (DIR)
- new net: R17.1, U4.4 (PORT)
- new net OVCUR_1: U1.27 (OVCUR1#), U16.3 (FLAG#)
- new net OVCUR_2: U1.29 (OVCUR2#), U17.3 (FLAG#)
- new net OVCUR_3: U1.31 (OVCUR3#/GANG_EN#), U18.3 (FLAG#)
- new net OVCUR_4: U1.33 (OVCUR4#/GANG_EN#), U19.3 (FLAG#)
- new net P3_SS_AC_TX+: C35.1, U3.6 (TXP)
- new net P3_SS_AC_TX-: C36.1, U3.7 (TXN)
- new net P3_SS_RX1+: J3.B11 (RX1+), U3.14 (RX1N), U5.1 (IO1)
- new net P3_SS_RX1-: J3.B10 (RX1-), U3.15 (RX1P), U5.2 (IO2)
- new net P4_SS_AC_TX+: C37.1, U4.6 (TXP)
- new net P4_SS_AC_TX-: C38.1, U4.7 (TXN)
- new net P4_SS_RX1+: J4.B11 (RX1+), U4.14 (RX1N), U7.5 (IO4)
- new net P4_SS_RX1-: J4.B10 (RX1-), U4.15 (RX1P), U7.4 (IO3)
- new net RESET: C30.1, R23.1, U1.46 (RESET#)
- new net UP_HS_AC_D+: J1.A6 (D+), J1.B6 (D+), U22.3 (I/O2)
- new net UP_HS_AC_D-: J1.A7 (D-), J1.B7 (D-), U22.1 (I/O1)
- new net UP_SS_AC_TX+: C39.1, U14.5 (IO4), U2.6 (TXP)
- new net UP_SS_AC_TX-: C40.1, U14.4 (IO3), U2.7 (TXN)
- new net UP_SS_RX1+: J1.B11 (RX1+), U2.14 (RX1N), U25.5 (IO4)
- new net UP_SS_RX1-: J1.B10 (RX1-), U2.15 (RX1P), U25.4 (IO3)
- new net UP_SS_RX2+: J1.A11 (RX2+), U2.19 (RX2P), U26.2 (IO2)
- new net UP_SS_RX2-: J1.A10 (RX2-), U2.18 (RX2N), U26.1 (IO1)
- new net UP_SS_TX1+: J1.A2 (TX1+), U2.16 (TX1N), U25.2 (IO2)
- new net UP_SS_TX1-: J1.A3 (TX1-), U2.17 (TX1P), U25.1 (IO1)
- new net UP_SS_TX2+: J1.B2 (TX2+), U2.21 (TX2P), U26.5 (IO4)
- new net UP_SS_TX2-: J1.B3 (TX2-), U2.20 (TX2N), U26.4 (IO3)
- no-connect marks 33 -> 35
Other:
- note added: "C16 can be bigger to prevent hub resets"
- note added: "GND on pins 2 and 4"
- note added: "TPD4E02B04DQA array"
- moved on the sheet: C16, C19, C21, C22, C23, C24, J3, J6, R3, R4, R5, R6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
